File: PCB/pico/musec_pico.kicad_sch (KiCad schematic)
At the start: 63 parts, among them J1 Pedal, J2 PJ313, J3 PJ313, SW1 SW_DIP_x01, SW2 SW_DIP_x01, SW3 SW_DIP_x01, SW4 SW_DIP_x01, SW5 SW_DIP_x01, SW6 SW_DIP_x01, SW7 SW_DIP_x01, U1 PiPico, U3 TMAG5273, U4 TMAG5273, U5 TMAG5273, U6 TMAG5273, U7 TMAG5273

Commit message: schematic rp2040 change
need to change power delivery/protection of usb lines, and also look over it again, add the schematic for the rp2040, and finish re-routing the PCB.
Parts:
- removed U1: PiPico, musec_pico:RPi_Pico_SMD_Pins, symbol musec_pico:PiPico
- added C11, C13, C14, C15, C16, C17, C19, C20, C21, C22, C23: 100nF, Capacitor_SMD:C_0402_1005Metric, symbol Device:C
- added C12, C18: 1uF, Capacitor_SMD:C_0402_1005Metric, symbol Device:C
- added C24, C25: 10uF, Capacitor_SMD:C_0805_2012Metric, symbol Device:C
- added CXTAL1, CXTAL2: 30pF, Capacitor_SMD:C_0402_1005Metric, symbol Device:C_Small
- added D23: SS34, Diode_SMD:D_SMA, symbol Device:D_Schottky
- added FU1: 0.5A, Fuse:Fuse_1206_3216Metric_Pad1.42x1.75mm_HandSolder, symbol Device:Fuse
- added R5: 1K, Resistor_SMD:R_0402_1005Metric, symbol Device:R
- added R6: 1K, Resistor_SMD:R_0603_1608Metric_Pad0.98x0.95mm_HandSolder, symbol Device:R
- added R7: 10K, Resistor_SMD:R_0603_1608Metric_Pad0.98x0.95mm_HandSolder, symbol Device:R
- added R8, R9: 27, Resistor_SMD:R_0603_1608Metric_Pad0.98x0.95mm_HandSolder, symbol Device:R
- added RV1, RV2: RL0603E005M500K, Resistor_SMD:R_0603_1608Metric_Pad0.98x0.95mm_HandSolder, symbol Device:Varistor
- added SWBOOT1: SW_Push, Button_Switch_THT:SW_PUSH_6mm_H4.3mm, symbol Switch:SW_Push
- added U2: RP2040, RP2040_minimal:RP2040-QFN-56, symbol MCU_RaspberryPi_RP2040:RP2040
- added UF1: W25Q128JVS, Package_SO:SOIC-8_5.275x5.275mm_P1.27mm, symbol Memory_Flash:W25Q128JVS
- added UV1: NCP1117-3.3_SOT223, Package_TO_SOT_SMD:SOT-223-3_TabPin2, symbol Regulator_Linear:NCP1117-3.3_SOT223
- added Y1: 12MHz, Crystal:Crystal_SMD_3225-4Pin_3.2x2.5mm, symbol Device:Crystal_GND24
Connections:
- net +3V3: now also C11.1, C12.1, C13.1, C14.1, C16.1, C19.1, C20.1, C21.1, C22.1, C23.1, C25.1, R7.1, U2.1 (IOVDD), U2.10 (IOVDD), U2.22 (IOVDD), U2.33 (IOVDD), U2.42 (IOVDD), U2.43 (ADC_AVDD), U2.44 (VREG_IN), U2.48 (USB_VDD), U2.49 (IOVDD), UF1.8 (VCC), UV1.2 (VO)
- net +5V: now also C24.1, D23.1 (K), UV1.3 (VI)
- net GND: now also C11.2, C12.2, C13.2, C14.2, C15.2, C16.2, C17.2, C18.2, C19.2, C20.2, C21.2, C22.2, C23.2, C24.2, C25.2, CXTAL1.1, CXTAL2.1, RV1.2, RV2.2, SWBOOT1.1, U2.19 (TESTEN), U2.57 (GND), UF1.4 (GND), UV1.1 (GND), Y1.2, Y1.4
- net K1: now also U2.27 (GPIO16)
- net K2: now also U2.28 (GPIO17)
- net K3: now also U2.29 (GPIO18)
- net K4: now also U2.30 (GPIO19)
- net K5: now also U2.31 (GPIO20)
- net K6: now also U2.32 (GPIO21)
- net K7: now also U2.34 (GPIO22)
- net SCL: now also U2.3 (GPIO1)
- net SDA: now also U2.2 (GPIO0)
- net VB1: now also U2.16 (GPIO13)
- net VB2: now also U2.15 (GPIO12)
- net VB3: now also U2.14 (GPIO11)
- net VB4: now also U2.13 (GPIO10)
- net VB5: now also U2.12 (GPIO9)
- net at USB1.11 (VBUS), USB1.2 (VBUS): now also FU1.2
- net USB_D-: now reaches USB1.5 (DN2), USB1.7 (DN1)
- net USB_D-: now also R9.1, RV2.1
- net USB_D+: now reaches USB1.6 (DP1), USB1.8 (DP2)
- net USB_D+: now also R8.1, RV1.1
- net LED: now reaches R3.2
- net LED: now also U2.17 (GPIO14)
- net PEDAL_BTN: now reaches J1.3 (Pin_3)
- net PEDAL_BTN: now also U2.5 (GPIO3)
- net RGB_PEDAL: now reaches R4.1
- net RGB_PEDAL: now also U2.18 (GPIO15)
- net TRS_PEDAL: now reaches J2.3 (T), J3.3 (T)
- net TRS_PEDAL: now also U2.6 (GPIO4)
- new net: R9.2, U2.46 (USB_DM)
- new net: R8.2, U2.47 (USB_DP)
- new net: CXTAL2.2, R5.2, Y1.3
- new net: D23.2 (A), FU1.1
- new net +1V1: C15.1, C17.1, C18.1, U2.23 (DVDD), U2.45 (VREG_VOUT), U2.50 (DVDD)
- new net GPIO2: U2.4 (GPIO2)
- new net GPIO28_ADC2: U2.40 (GPIO28_ADC2)
- new net GPIO29_ADC3: U2.41 (GPIO29_ADC3)
- new net QSPI_SCLK: U2.52 (QSPI_SCLK), UF1.6 (CLK)
- new net QSPI_SD0: U2.53 (QSPI_SD0), UF1.5 (DI(IO0))
- new net QSPI_SD1: U2.55 (QSPI_SD1), UF1.2 (DO(IO1))
- new net QSPI_SD2: U2.54 (QSPI_SD2), UF1.3 (IO2)
- new net QSPI_SD3: U2.51 (QSPI_SD3), UF1.7 (IO3)
- new net QSPI_SS: R6.1, R7.2, U2.56 (QSPI_SS), UF1.1 (~{CS})
- new net RUN: U2.26 (RUN)
- new net SWCLK: U2.24 (SWCLK)
- new net SWDIO: U2.25 (SWD)
- new net XIN: CXTAL1.2, U2.20 (XIN), Y1.1
- new net XOUT: R5.1, U2.21 (XOUT)
- new net ~{USB_BOOT}: R6.2, SWBOOT1.2
- no-connect marks 18 -> 8
Other:
- note added: "1.1V Smoothing"
- note added: "12MHz, 20pF"
- note added: "3.3V Smoothing"
- note added: "30pF/2 + stray capacitance of 5pF = 20pF"
- note added: "C4 - Close to pin 45 of RP2040"
- note added: "C8 - Close to pin 44 of rp2040"
- note added: "Crystal"
- note added: "Crystal & Code Storage"
- note added: "Debug"
- note added: "Diff pair of .5mm"
- note added: "Flash"
- note added: "Flash Chip"
- note added: "PWR"
- note added: "Pedal Connector"
- note added: "Power for RP2040"
- note added: "RP2040 Interfaces"
- note added: "Stepdown to 3.3v"
- note added: "ULCE1005A015FR"
- note added: "USB/PWR In"
- note added: "fix this (later) ((its old method))"
- moved on the sheet: C10, C6, C7, C8, C9, R4
